File: NRF24-breakout.kicad_pcb (KiCad board)
At the start: 2 copper layers, 0 parts

Commit message: Edge cut
Parts:
- added J1: CONN_01X08, Pin_Headers:Pin_Header_Straight_1x08_Pitch2.54mm, F.Cu at (153.6, 117.6)
- added U1: nRF24, nRF24-footprints:nRF24, F.Cu at (144.1, 127.0)
Other:
- board outline added: 27.3 x 22.9 mm
- rule pad_to_mask_clearance: 0.2 -> 0
Changed lines of the file:
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@@
 (kicad_pcb (version 4) (host pcbnew 4.0.6)
   (general
-    (links 0)
-    (no_connects 0)
+    (links 7)
+    (no_connects 7)
     (area 0 0 0 0)
     (thickness 1.6)
-    (drawings 0)
+    (drawings 4)
     (tracks 0)
     (zones 0)
-    (modules 0)
-    (nets 1)
+    (modules 2)
+    (nets 9)
   )
   (page A4)
-  (title_block
-    (title "nRF24 Breakout")
-    (date 2017-08-11)
-    (rev 1.0)
-    (company UnlikeNoise)
-    (comment 1 "Leon van Bokhorst")
-  )
   (layers
     (0 F.Cu signal)
@@
     (trace_min 0.2)
     (segment_width 0.2)
-    (edge_width 0.15)
+    (edge_width 0.1)
     (via_size 0.6)
     (via_drill 0.4)
@@
     (mod_text_size 1 1)
     (mod_text_width 0.15)
-    (pad_size 1.524 1.524)
-    (pad_drill 0.762)
-    (pad_to_mask_clearance 0.2)
+    (pad_size 1.5 1.5)
+    (pad_drill 0.6)
+    (pad_to_mask_clearance 0)
     (aux_axis_origin 0 0)
     (visible_elements FFFFFF7F)
@@
   )
   (net 0 "")
+  (net 1 "Net-(J1-Pad1)")
+  (net 2 "Net-(J1-Pad2)")
+  (net 3 "Net-(J1-Pad3)")
+  (net 4 "Net-(J1-Pad4)")
+  (net 5 "Net-(J1-Pad5)")
+  (net 6 "Net-(J1-Pad6)")
+  (net 7 "Net-(J1-Pad7)")
+  (net 8 "Net-(J1-Pad8)")
   (net_class Default "This is the default net class."
     (clearance 0.2)
@@
     (uvia_dia 0.3)
     (uvia_drill 0.1)
-  )
+    (add_net "Net-(J1-Pad1)")
+    (add_net "Net-(J1-Pad2)")
+    (add_net "Net-(J1-Pad3)")
+    (add_net "Net-(J1-Pad4)")
+    (add_net "Net-(J1-Pad5)")
+    (add_net "Net-(J1-Pad6)")
+    (add_net "Net-(J1-Pad7)")
+    (add_net "Net-(J1-Pad8)")
+  )
+  (module Pin_Headers:Pin_Header_Straight_1x08_Pitch2.54mm (layer F.Cu)
+    (at 153.623333 117.605)
+    (descr "Through hole straight pin header, 1x08, 2.54mm pitch, single row")
+    (tags "Through hole pin header THT 1x08 2.54mm single row")
+    (fp_text reference J1 (at 0 -2.33) (layer F.SilkS)
+      (effects (font (size 1 1) (thickness 0.15)))
+    )
+    (fp_text value CONN_01X08 (at 0 20.11) (layer F.Fab)
+      (effects (font (size 1 1) (thickness 0.15)))
+    )
+    (fp_line (start -0.635 -1.27) (end 1.27 -1.27) (layer F.Fab) (width 0.1))
+    (fp_line (start 1.27 -1.27) (end 1.27 19.05) (layer F.Fab) (width 0.1))
+    (fp_line (start 1.27 19.05) (end -1.27 19.05) (layer F.Fab) (width 0.1))
+    (fp_line (start -1.27 19.05) (end -1.27 -0.635) (layer F.Fab) (width 0.1))
+    (fp_line (start -1.27 -0.635) (end -0.635 -1.27) (layer F.Fab) (width 0.1))
+    (fp_line (start -1.33 19.11) (end 1.33 19.11) (layer F.SilkS) (width 0.12))
+    (fp_line (start -1.33 1.27) (end -1.33 19.11) (layer F.SilkS) (width 0.12))
+    (fp_line (start 1.33 1.27) (end 1.33 19.11) (layer F.SilkS) (width 0.12))
+    (fp_line (start -1.33 1.27) (end 1.33 1.27) (layer F.SilkS) (width 0.12))
+    (fp_line (start -1.33 0) (end -1.33 -1.33) (layer F.SilkS) (width 0.12))
+    (fp_line (start -1.33 -1.33) (end 0 -1.33) (layer F.SilkS) (width 0.12))
+    (fp_line (start -1.8 -1.8) (end -1.8 19.55) (layer F.CrtYd) (width 0.05))
+    (fp_line (start -1.8 19.55) (end 1.8 19.55) (layer F.CrtYd) (width 0.05))
+    (fp_line (start 1.8 19.55) (end 1.8 -1.8) (layer F.CrtYd) (width 0.05))
+    (fp_line (start 1.8 -1.8) (end -1.8 -1.8) (layer F.CrtYd) (width 0.05))
+    (fp_text user %R (at 0 8.89 90) (layer F.Fab)
+      (effects (font (size 1 1) (thickness 0.15)))
+    )
+    (pad 1 thru_hole rect (at 0 0) (size 1.7 1.7) (drill 1) (layers *.Cu *.Mask)
+      (net 1 "Net-(J1-Pad1)"))
+    (pad 2 thru_hole oval (at 0 2.54) (size 1.7 1.7) (drill 1) (layers *.Cu *.Mask)
+      (net 2 "Net-(J1-Pad2)"))
+    (pad 3 thru_hole oval (at 0 5.08) (size 1.7 1.7) (drill 1) (layers *.Cu *.Mask)
+      (net 3 "Net-(J1-Pad3)"))
+    (pad 4 thru_hole oval (at 0 7.62) (size 1.7 1.7) (drill 1) (layers *.Cu *.Mask)
+      (net 4 "Net-(J1-Pad4)"))
+    (pad 5 thru_hole oval (at 0 10.16) (size 1.7 1.7) (drill 1) (layers *.Cu *.Mask)
+      (net 5 "Net-(J1-Pad5)"))
+    (pad 6 thru_hole oval (at 0 12.7) (size 1.7 1.7) (drill 1) (layers *.Cu *.Mask)
+      (net 6 "Net-(J1-Pad6)"))
+    (pad 7 thru_hole oval (at 0 15.24) (size 1.7 1.7) (drill 1) (layers *.Cu *.Mask)
+      (net 7 "Net-(J1-Pad7)"))
+    (pad 8 thru_hole oval (at 0 17.78) (size 1.7 1.7) (drill 1) (layers *.Cu *.Mask)
+      (net 8 "Net-(J1-Pad8)"))
+    (model ${KISYS3DMOD}/Pin_Headers.3dshapes/Pin_Header_Straight_1x08_Pitch2.54mm.wrl
+      (at (xyz 0 0 0))
+      (scale (xyz 1 1 1))
+      (rotate (xyz 0 0 0))
+    )
+  )
+  (module nRF24-footprints:nRF24 (layer F.Cu)
+    (at 144.145 127)
+    (descr "A footprint for the generic nRF24 module")
+    (fp_text reference U1 (at -10.16 2.54) (layer F.SilkS)
+      (effects (font (size 1 1) (thickness 0.15)))
+    )
+    (fp_text value nRF24 (at -10.16 -5.08) (layer F.Fab)
+      (effects (font (size 1 1) (thickness 0.15)))
+    )
+    (fp_line (start -13.97 4.445) (end 5.08 4.445) (layer F.SilkS) (width 0.15))
+    (fp_line (start -13.97 4.445) (end -13.97 -6.985) (layer F.SilkS) (width 0.15))
+    (fp_line (start 5.08 4.445) (end -13.97 4.445) (layer F.SilkS) (width 0.15))
+    (fp_line (start 5.08 4.445) (end 5.08 -6.985) (layer F.SilkS) (width 0.15))
+    (fp_line (start 5.08 -6.985) (end 5.08 4.445) (layer F.SilkS) (width 0.15))
+    (fp_line (start 5.08 -6.985) (end -13.97 -6.985) (layer F.SilkS) (width 0.15))
+    (fp_text user Vcc (at -1.27 2.54 90) (layer F.SilkS)
+      (effects (font (size 0.5 0.5) (thickness 0.125)))
+    )
+    (fp_text user CSN (at -1.27 0 90) (layer F.SilkS)
+      (effects (font (size 0.5 0.5) (thickness 0.125)))
+    )
+    (fp_text user MOSI (at -1.27 -2.54 90) (layer F.SilkS)
+      (effects (font (size 0.5 0.5) (thickness 0.125)))
+    )
+    (fp_text user IRQ (at -1.27 -5.08 90) (layer F.SilkS)
+      (effects (font (size 0.5 0.5) (thickness 0.125)))
+    )
+    (fp_text user SCK (at 3.81 -2.54 90) (layer F.SilkS)
+      (effects (font (size 0.5 0.5) (thickness 0.125)))
+    )
+    (fp_text user MISO (at 3.81 -5.08 90) (layer F.SilkS)
+      (effects (font (size 0.5 0.5) (thickness 0.125)))
+    )
+    (fp_text user CE (at 3.81 0 90) (layer F.SilkS)
+      (effects (font (size 0.5 0.5) (thickness 0.125)))
+    )
+    (fp_text user GND (at 3.81 2.54 90) (layer F.SilkS)
+      (effects (font (size 0.5 0.5) (thickness 0.125)))
+    )
+    (pad 2 thru_hole circle (at 2.54 -2.54) (size 1.524 1.524) (drill 0.762) (layers *.Cu *.Mask)
+      (net 3 "Net-(J1-Pad3)"))
+    (pad 0 thru_hole circle (at 2.54 2.54) (size 1.524 1.524) (drill 0.762) (layers *.Cu *.Mask)
+      (net 1 "Net-(J1-Pad1)"))
+    (pad 1 thru_hole circle (at 2.54 0) (size 1.524 1.524) (drill 0.762) (layers *.Cu *.Mask)
+      (net 2 "Net-(J1-Pad2)"))
+    (pad 18 thru_hole circle (at 0 2.54) (size 1.524 1.524) (drill 0.762) (layers *.Cu *.Mask))
+    (pad 6 thru_hole circle (at 0 0) (size 1.524 1.524) (drill 0.762) (layers *.Cu *.Mask)
+      (net 7 "Net-(J1-Pad7)"))
+    (pad 5 thru_hole circle (at 0 -2.54) (size 1.524 1.524) (drill 0.762) (layers *.Cu *.Mask)
+      (net 6 "Net-(J1-Pad6)"))
+    (pad 4 thru_hole circle (at 0 -5.08) (size 1.524 1.524) (drill 0.762) (layers *.Cu *.Mask)
+      (net 5 "Net-(J1-Pad5)"))
+    (pad 3 thru_hole circle (at 2.54 -5.08) (size 1.524 1.524) (drill 0.762) (layers *.Cu *.Mask)
+      (net 4 "Net-(J1-Pad4)"))
+  )
+  (gr_line (start 128.905 137.795) (end 156.21 137.795) (angle 90) (layer Edge.Cuts) (width 0.1))
+  (gr_line (start 128.905 114.935) (end 128.905 137.795) (angle 90) (layer Edge.Cuts) (width 0.1))
+  (gr_line (start 156.21 114.935) (end 128.905 114.935) (angle 90) (layer Edge.Cuts) (width 0.1))
+  (gr_line (start 156.21 137.795) (end 156.21 114.935) (angle 90) (layer Edge.Cuts) (width 0.1))
 )

Commit message: Wiring
Parts:
- moved J1 0.14 mm to (153.7, 117.5)
Routing:
- net Net-(J1-Pad1): track 0.00 -> 28.4 mm
- net Net-(J1-Pad2): track 0.00 -> 23.5 mm
- net Net-(J1-Pad3): track 0.00 -> 19.5 mm
- net Net-(J1-Pad6): track 0.00 -> 13.8 mm
- net Net-(J1-Pad5): track 0.00 -> 12.1 mm
- net Net-(J1-Pad7): track 0.00 -> 11.9 mm
- net Net-(J1-Pad8): track 0.00 -> 11.9 mm
- net Net-(J1-Pad4): track 0.00 -> 9.04 mm
Changed lines of the file:
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@@
 (kicad_pcb (version 4) (host pcbnew 4.0.6)
   (general
-    (links 7)
-    (no_connects 7)
-    (area 0 0 0 0)
+    (links 8)
+    (no_connects 0)
+    (area 128.854999 114.884999 158.703334 138.66)
     (thickness 1.6)
     (drawings 4)
-    (tracks 0)
+    (tracks 55)
     (zones 0)
     (modules 2)
@@
   )
   (page A4)
+  (title_block
+    (title "nRF24 Breakout")
+    (date 2017-03-11)
+    (rev 1.0)
+    (company UnlikeNoise)
+    (comment 1 "Leon van Bokhorst")
+  )
   (layers
     (0 F.Cu signal)
@@
     (mod_text_size 1 1)
     (mod_text_width 0.15)
-    (pad_size 1.5 1.5)
-    (pad_drill 0.6)
+    (pad_size 1.524 1.524)
+    (pad_drill 0.762)
     (pad_to_mask_clearance 0)
     (aux_axis_origin 0 0)
@@
   )
   (module Pin_Headers:Pin_Header_Straight_1x08_Pitch2.54mm (layer F.Cu)
-    (at 153.623333 117.605)
+    (at 153.67 117.475)
     (descr "Through hole straight pin header, 1x08, 2.54mm pitch, single row")
     (tags "Through hole pin header THT 1x08 2.54mm single row")
-    (fp_text reference J1 (at 0 -2.33) (layer F.SilkS)
-      (effects (font (size 1 1) (thickness 0.15)))
-    )
-    (fp_text value CONN_01X08 (at 0 20.11) (layer F.Fab)
+    (fp_text reference J1 (at -3.128333 -0.765) (layer F.SilkS)
+      (effects (font (size 1 1) (thickness 0.15)))
+    )
+    (fp_text value CONN_01X08 (at 0 20.11) (layer F.Fab) hide
       (effects (font (size 1 1) (thickness 0.15)))
     )
@@
     (at 144.145 127)
     (descr "A footprint for the generic nRF24 module")
-    (fp_text reference U1 (at -10.16 2.54) (layer F.SilkS)
-      (effects (font (size 1 1) (thickness 0.15)))
-    )
-    (fp_text value nRF24 (at -10.16 -5.08) (layer F.Fab)
+    (fp_text reference U1 (at -3.81 5.715) (layer F.SilkS)
+      (effects (font (size 1 1) (thickness 0.15)))
+    )
+    (fp_text value nRF24 (at -6.35 -1.27) (layer F.Fab)
       (effects (font (size 1 1) (thickness 0.15)))
     )
@@
     (pad 1 thru_hole circle (at 2.54 0) (size 1.524 1.524) (drill 0.762) (layers *.Cu *.Mask)
       (net 2 "Net-(J1-Pad2)"))
-    (pad 18 thru_hole circle (at 0 2.54) (size 1.524 1.524) (drill 0.762) (layers *.Cu *.Mask))
+    (pad 7 thru_hole circle (at 0 2.54) (size 1.524 1.524) (drill 0.762) (layers *.Cu *.Mask)
+      (net 8 "Net-(J1-Pad8)"))
     (pad 6 thru_hole circle (at 0 0) (size 1.524 1.524) (drill 0.762) (layers *.Cu *.Mask)
       (net 7 "Net-(J1-Pad7)"))
@@
   (gr_line (start 156.21 114.935) (end 128.905 114.935) (angle 90) (layer Edge.Cuts) (width 0.1))
   (gr_line (start 156.21 137.795) (end 156.21 114.935) (angle 90) (layer Edge.Cuts) (width 0.1))
+  (segment (start 146.685 129.54) (end 146.05 129.54) (width 0.25) (layer F.Cu) (net 1))
+  (segment (start 146.05 129.54) (end 144.78 128.27) (width 0.25) (layer F.Cu) (net 1))
+  (segment (start 144.78 128.27) (end 142.24 128.27) (width 0.25) (layer F.Cu) (net 1))
+  (segment (start 142.875 117.475) (end 153.67 117.475) (width 0.25) (layer F.Cu) (net 1))
+  (segment (start 142.24 118.11) (end 142.875 117.475) (width 0.25) (layer F.Cu) (net 1))
+  (segment (start 140.335 120.015) (end 142.24 118.11) (width 0.25) (layer F.Cu) (net 1))
+  (segment (start 140.335 126.365) (end 140.335 120.015) (width 0.25) (layer F.Cu) (net 1))
+  (segment (start 142.24 128.27) (end 140.335 126.365) (width 0.25) (layer F.Cu) (net 1))
+  (segment (start 146.685 127) (end 146.05 127) (width 0.25) (layer F.Cu) (net 2))
+  (segment (start 146.05 127) (end 144.78 125.73) (width 0.25) (layer F.Cu) (net 2))
+  (segment (start 151.13 120.015) (end 153.67 120.015) (width 0.25) (layer F.Cu) (net 2))
+  (segment (start 150.495 119.38) (end 151.13 120.015) (width 0.25) (layer F.Cu) (net 2))
+  (segment (start 142.24 119.38) (end 150.495 119.38) (width 0.25) (layer F.Cu) (net 2))
+  (segment (start 141.605 120.015) (end 142.24 119.38) (width 0.25) (layer F.Cu) (net 2))
+  (segment (start 141.605 125.095) (end 141.605 120.015) (width 0.25) (layer F.Cu) (net 2))
+  (segment (start 142.24 125.73) (end 141.605 125.095) (width 0.25) (layer F.Cu) (net 2))
+  (segment (start 144.78 125.73) (end 142.24 125.73) (width 0.25) (layer F.Cu) (net 2))
+  (segment (start 146.685 124.46) (end 145.796 124.46) (width 0.25) (layer F.Cu) (net 3))
+  (segment (start 151.765 122.555) (end 153.67 122.555) (width 0.25) (layer F.Cu) (net 3))
+  (segment (start 149.606 120.396) (end 151.765 122.555) (width 0.25) (layer F.Cu) (net 3))
+  (segment (start 142.748 120.396) (end 149.606 120.396) (width 0.25) (layer F.Cu) (net 3))
+  (segment (start 142.24 120.904) (end 142.748 120.396) (width 0.25) (layer F.Cu) (net 3))
+  (segment (start 142.24 122.682) (end 142.24 120.904) (width 0.25) (layer F.Cu) (net 3))
+  (segment (start 142.748 123.19) (end 142.24 122.682) (width 0.25) (layer F.Cu) (net 3))
+  (segment (start 143.256 123.19) (end 142.748 123.19) (width 0.25) (layer F.Cu) (net 3))
+  (segment (start 144.526 123.19) (end 143.256 123.19) (width 0.25) (layer F.Cu) (net 3))
+  (segment (start 145.796 124.46) (end 144.526 123.19) (width 0.25) (layer F.Cu) (net 3))
+  (segment (start 151.765 125.095) (end 153.67 125.095) (width 0.25) (layer F.Cu) (net 4))
+  (segment (start 150.495 123.825) (end 151.765 125.095) (width 0.25) (layer F.Cu) (net 4))
+  (segment (start 150.495 122.555) (end 150.495 123.825) (width 0.25) (layer F.Cu) (net 4))
+  (segment (start 149.86 121.92) (end 150.495 122.555) (width 0.25) (layer F.Cu) (net 4))
+  (segment (start 146.685 121.92) (end 149.86 121.92) (width 0.25) (layer F.Cu) (net 4))
+  (segment (start 151.638 126.238) (end 152.273 126.238) (width 0.25) (layer F.Cu) (net 5))
+  (segment (start 152.273 126.238) (end 153.67 127.635) (width 0.25) (layer F.Cu) (net 5))
+  (segment (start 144.145 121.92) (end 145.415 123.19) (width 0.25) (layer F.Cu) (net 5))
+  (segment (start 148.59 123.19) (end 151.638 126.238) (width 0.25) (layer F.Cu) (net 5))
+  (segment (start 151.638 126.238) (end 151.765 126.365) (width 0.25) (layer F.Cu) (net 5))
+  (segment (start 145.415 123.19) (end 148.59 123.19) (width 0.25) (layer F.Cu) (net 5))
+  (segment (start 146.05 125.73) (end 145.796 125.476) (width 0.25) (layer F.Cu) (net 6))
+  (segment (start 153.67 130.175) (end 151.13 130.175) (width 0.25) (layer F.Cu) (net 6))
+  (segment (start 150.495 129.54) (end 151.13 130.175) (width 0.25) (layer F.Cu) (net 6))
+  (segment (start 150.495 126.365) (end 150.495 129.54) (width 0.25) (layer F.Cu) (net 6))
+  (segment (start 149.86 125.73) (end 150.495 126.365) (width 0.25) (layer F.Cu) (net 6))
+  (segment (start 146.05 125.73) (end 149.86 125.73) (width 0.25) (layer F.Cu) (net 6))
+  (segment (start 145.796 125.476) (end 144.78 124.46) (width 0.25) (layer F.Cu) (net 6))
+  (segment (start 144.145 124.46) (end 144.78 124.46) (width 0.25) (layer F.Cu) (net 6))
+  (segment (start 151.13 131.445) (end 152.4 131.445) (width 0.25) (layer F.Cu) (net 7))
+  (segment (start 147.955 128.27) (end 151.13 131.445) (width 0.25) (layer F.Cu) (net 7))
+  (segment (start 146.05 128.27) (end 147.955 128.27) (width 0.25) (layer F.Cu) (net 7))
+  (segment (start 144.78 127) (end 146.05 128.27) (width 0.25) (layer F.Cu) (net 7))
+  (segment (start 152.4 131.445) (end 153.67 132.715) (width 0.25) (layer F.Cu) (net 7))
+  (segment (start 144.145 127) (end 144.78 127) (width 0.25) (layer F.Cu) (net 7))
+  (segment (start 144.145 129.54) (end 144.526 129.54) (width 0.25) (layer F.Cu) (net 8))
+  (segment (start 144.526 129.54) (end 150.241 135.255) (width 0.25) (layer F.Cu) (net 8))
+  (segment (start 150.241 135.255) (end 153.67 135.255) (width 0.25) (layer F.Cu) (net 8))
 )

Commit message: Labels
Other:
- board text added: "CE"
- board text added: "CSN"
- board text added: "GND"
- board text added: "IRQ"
- board text added: "MISO"
- board text added: "MOSI"
- board text added: "SCK"
- board text added: "UnlikeNoise nRF24 version 1.0"
- board text added: "Vcc"
Changed lines of the file:
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@@
     (links 8)
     (no_connects 0)
-    (area 128.854999 114.884999 158.703334 138.66)
+    (area 128.854999 114.884999 156.260001 137.845001)
     (thickness 1.6)
-    (drawings 4)
+    (drawings 13)
     (tracks 55)
     (zones 0)
@@
     (descr "Through hole straight pin header, 1x08, 2.54mm pitch, single row")
     (tags "Through hole pin header THT 1x08 2.54mm single row")
-    (fp_text reference J1 (at -3.128333 -0.765) (layer F.SilkS)
+    (fp_text reference J1 (at -2.54 -1.651) (layer F.SilkS)
       (effects (font (size 1 1) (thickness 0.15)))
     )
@@
       (net 4 "Net-(J1-Pad4)"))
   )
+  (gr_text "UnlikeNoise nRF24 version 1.0" (at 138.938 135.636) (layer F.SilkS)
+    (effects (font (size 0.4 0.4) (thickness 0.1)))
+  )
+  (gr_text GND (at 151.13 117.348) (layer F.SilkS)
+    (effects (font (size 0.6 0.6) (thickness 0.15)))
+  )
+  (gr_text CE (at 151.13 119.888) (layer F.SilkS)
+    (effects (font (size 0.6 0.6) (thickness 0.15)))
+  )
+  (gr_text SCK (at 151.13 122.428) (layer F.SilkS)
+    (effects (font (size 0.6 0.6) (thickness 0.15)))
+  )
+  (gr_text MISO (at 151.13 124.968) (layer F.SilkS)
+    (effects (font (size 0.6 0.6) (thickness 0.15)))
+  )
+  (gr_text IRQ (at 151.13 127.508) (layer F.SilkS)
+    (effects (font (size 0.6 0.6) (thickness 0.15)))
+  )
+  (gr_text MOSI (at 151.13 130.048) (layer F.SilkS)
+    (effects (font (size 0.6 0.6) (thickness 0.15)))
+  )
+  (gr_text CSN (at 151.13 132.588) (layer F.SilkS)
+    (effects (font (size 0.6 0.6) (thickness 0.15)))
+  )
+  (gr_text Vcc (at 151.13 135.128) (layer F.SilkS)
+    (effects (font (size 0.6 0.6) (thickness 0.15)))
+  )
   (gr_line (start 128.905 137.795) (end 156.21 137.795) (angle 90) (layer Edge.Cuts) (width 0.1))

Commit message: Update Pcbnew with the new netlist
Parts:
- added C1: 10uF, Capacitors_THT:CP_Radial_D10.0mm_P5.00mm, F.Cu at (142.2, 137.7)
Routing:
- net Net-(C1-Pad1): track 11.9 -> 20.8 mm
Other:
- board size 27.3 x 22.9 mm -> 27.3 x 30.4 mm
- board text added: "UnlikeNoise nRF24 v1.01"
- board text removed: "UnlikeNoise nRF24 version 1.0"
